File: sichergo/sichergo.kicad_pcb (KiCad board)
At the start: 2 copper layers, 97 parts, among them J1 Conn_01x04_Pin, J2 Conn_01x04_Pin, SW1 SW_Push, SW10 SW_Push, SW11 SW_Push, SW12 SW_Push, SW13 SW_Push, SW14 SW_Push, SW15 SW_Push, SW16 SW_Push, SW17 SW_Push, SW18 SW_Push, SW19 SW_Push, SW20 SW_Push, SW21 SW_Push, SW22 SW_Push, SW23 SW_Push, SW24 SW_Push, SW25 SW_Push, SW26 SW_Push, SW27 SW_Push, SW28 SW_Push, SW29 SW_Push, SW3 SW_Push, SW30 SW_Push, SW31 SW_Push, SW32 SW_Push, SW33 SW_Push, SW34 SW_Push, SW35 SW_Push, SW36 SW_Push, SW37 SW_Push, SW4 SW_Push, SW5 SW_Push, SW6 SW_Push, SW7 SW_Push, SW8 SW_Push, SW9 SW_Push, U1 AZ1117-3.3, U10 SN74LVC1G125DBV, U2 TPD4E05U06DQA, U3 YTS1C0033BBG01, U4 STM32F103C8Tx, U5 SN74LVC1G125DBV, U6 SN74LVC1G125DBV, U7 YTS1C0033BBG01, U8 STM32F103C8Tx, U9 SN74LVC1G125DBV, Y1 Crystal_GND24, Y2 Crystal_GND24

Commit message: Start layout
Parts:
- added D38: LED, LED_SMD:LED_0603_1608Metric_Pad1.05x0.95mm_HandSolder, F.Cu at (216.8, -78.2)
- added D39: LED, LED_SMD:LED_0603_1608Metric_Pad1.05x0.95mm_HandSolder, F.Cu at (216.8, -75.6)
- added D40: LED, LED_SMD:LED_0603_1608Metric_Pad1.05x0.95mm_HandSolder, F.Cu at (216.8, -73.0)
- added D41: LED, LED_SMD:LED_0603_1608Metric_Pad1.05x0.95mm_HandSolder, F.Cu at (216.8, -70.4)
- added D42: LED, LED_SMD:LED_0603_1608Metric_Pad1.05x0.95mm_HandSolder, F.Cu at (216.8, -67.8)
- added D43: LED, LED_SMD:LED_0603_1608Metric_Pad1.05x0.95mm_HandSolder, F.Cu at (216.8, -65.2)
- added D44: LED, LED_SMD:LED_0603_1608Metric_Pad1.05x0.95mm_HandSolder, F.Cu at (216.8, -62.6)
- added D45: LED, LED_SMD:LED_0603_1608Metric_Pad1.05x0.95mm_HandSolder, F.Cu at (221.2, -78.2)
- added D46: LED, LED_SMD:LED_0603_1608Metric_Pad1.05x0.95mm_HandSolder, F.Cu at (221.2, -75.6)
- added D47: LED, LED_SMD:LED_0603_1608Metric_Pad1.05x0.95mm_HandSolder, F.Cu at (221.2, -73.0)
- added D48: LED, LED_SMD:LED_0603_1608Metric_Pad1.05x0.95mm_HandSolder, F.Cu at (221.2, -70.4)
- added D49: LED, LED_SMD:LED_0603_1608Metric_Pad1.05x0.95mm_HandSolder, F.Cu at (221.2, -67.8)
- added D50: LED, LED_SMD:LED_0603_1608Metric_Pad1.05x0.95mm_HandSolder, F.Cu at (221.2, -65.2)
- added D51: LED, LED_SMD:LED_0603_1608Metric_Pad1.05x0.95mm_HandSolder, F.Cu at (221.2, -62.6)
- added D52: LED, LED_SMD:LED_0603_1608Metric_Pad1.05x0.95mm_HandSolder, F.Cu at (225.6, -78.2)
- added D53: LED, LED_SMD:LED_0603_1608Metric_Pad1.05x0.95mm_HandSolder, F.Cu at (225.6, -75.6)
- added D54: LED, LED_SMD:LED_0603_1608Metric_Pad1.05x0.95mm_HandSolder, F.Cu at (225.6, -73.0)
- added D55: LED, LED_SMD:LED_0603_1608Metric_Pad1.05x0.95mm_HandSolder, F.Cu at (225.6, -70.4)
- added D56: LED, LED_SMD:LED_0603_1608Metric_Pad1.05x0.95mm_HandSolder, F.Cu at (216.8, -58.0)
- added D57: LED, LED_SMD:LED_0603_1608Metric_Pad1.05x0.95mm_HandSolder, F.Cu at (216.8, -55.4)
- added D58: LED, LED_SMD:LED_0603_1608Metric_Pad1.05x0.95mm_HandSolder, F.Cu at (216.8, -52.8)
- added D59: LED, LED_SMD:LED_0603_1608Metric_Pad1.05x0.95mm_HandSolder, F.Cu at (216.8, -50.2)
- added D60: LED, LED_SMD:LED_0603_1608Metric_Pad1.05x0.95mm_HandSolder, F.Cu at (216.8, -47.7)
- added D61: LED, LED_SMD:LED_0603_1608Metric_Pad1.05x0.95mm_HandSolder, F.Cu at (216.8, -45.1)
- added D62: LED, LED_SMD:LED_0603_1608Metric_Pad1.05x0.95mm_HandSolder, F.Cu at (216.8, -42.5)
- added D63: LED, LED_SMD:LED_0603_1608Metric_Pad1.05x0.95mm_HandSolder, F.Cu at (221.2, -58.0)
- added D64: LED, LED_SMD:LED_0603_1608Metric_Pad1.05x0.95mm_HandSolder, F.Cu at (221.2, -55.4)
- added D65: LED, LED_SMD:LED_0603_1608Metric_Pad1.05x0.95mm_HandSolder, F.Cu at (221.2, -52.8)
- added D66: LED, LED_SMD:LED_0603_1608Metric_Pad1.05x0.95mm_HandSolder, F.Cu at (221.2, -50.2)
- added D67: LED, LED_SMD:LED_0603_1608Metric_Pad1.05x0.95mm_HandSolder, F.Cu at (221.2, -47.7)
- added D68: LED, LED_SMD:LED_0603_1608Metric_Pad1.05x0.95mm_HandSolder, F.Cu at (221.2, -45.1)
- added D69: LED, LED_SMD:LED_0603_1608Metric_Pad1.05x0.95mm_HandSolder, F.Cu at (221.2, -42.5)
- added D70: LED, LED_SMD:LED_0603_1608Metric_Pad1.05x0.95mm_HandSolder, F.Cu at (225.6, -58.0)
- added D71: LED, LED_SMD:LED_0603_1608Metric_Pad1.05x0.95mm_HandSolder, F.Cu at (225.6, -55.4)
- added D72: LED, LED_SMD:LED_0603_1608Metric_Pad1.05x0.95mm_HandSolder, F.Cu at (225.6, -52.8)
- added D73: LED, LED_SMD:LED_0603_1608Metric_Pad1.05x0.95mm_HandSolder, F.Cu at (225.6, -50.2)
- added Q1: 2N7002, Package_TO_SOT_SMD:SOT-23_Handsoldering, F.Cu at (246.1, -56.8)
- added Q2: 2N7002, Package_TO_SOT_SMD:SOT-23_Handsoldering, F.Cu at (246.1, -76.9)
- added R15: 1 kohm, Resistor_SMD:R_0603_1608Metric_Pad0.98x0.95mm_HandSolder, F.Cu at (230.0, -78.2)
- added R16: 1 kohm, Resistor_SMD:R_0603_1608Metric_Pad0.98x0.95mm_HandSolder, F.Cu at (230.0, -75.7)
- added R17: 1 kohm, Resistor_SMD:R_0603_1608Metric_Pad0.98x0.95mm_HandSolder, F.Cu at (230.0, -73.2)
- added R18: 1 kohm, Resistor_SMD:R_0603_1608Metric_Pad0.98x0.95mm_HandSolder, F.Cu at (230.0, -70.7)
- added R19: 1 kohm, Resistor_SMD:R_0603_1608Metric_Pad0.98x0.95mm_HandSolder, F.Cu at (230.0, -68.2)
- added R20: 1 kohm, Resistor_SMD:R_0603_1608Metric_Pad0.98x0.95mm_HandSolder, F.Cu at (230.0, -65.6)
- added R21: 1 kohm, Resistor_SMD:R_0603_1608Metric_Pad0.98x0.95mm_HandSolder, F.Cu at (230.0, -63.1)
- added R22: 1 kohm, Resistor_SMD:R_0603_1608Metric_Pad0.98x0.95mm_HandSolder, F.Cu at (234.3, -78.2)
- added R23: 1 kohm, Resistor_SMD:R_0603_1608Metric_Pad0.98x0.95mm_HandSolder, F.Cu at (234.3, -75.7)
- added R24: 1 kohm, Resistor_SMD:R_0603_1608Metric_Pad0.98x0.95mm_HandSolder, F.Cu at (234.3, -73.2)
- added R25: 1 kohm, Resistor_SMD:R_0603_1608Metric_Pad0.98x0.95mm_HandSolder, F.Cu at (234.3, -70.7)
- added R26: 1 kohm, Resistor_SMD:R_0603_1608Metric_Pad0.98x0.95mm_HandSolder, F.Cu at (234.3, -68.2)
- added R27: 1 kohm, Resistor_SMD:R_0603_1608Metric_Pad0.98x0.95mm_HandSolder, F.Cu at (234.3, -65.6)
- added R28: 1 kohm, Resistor_SMD:R_0603_1608Metric_Pad0.98x0.95mm_HandSolder, F.Cu at (234.3, -63.1)
- added R29: 1 kohm, Resistor_SMD:R_0603_1608Metric_Pad0.98x0.95mm_HandSolder, F.Cu at (238.7, -78.2)
- added R30: 1 kohm, Resistor_SMD:R_0603_1608Metric_Pad0.98x0.95mm_HandSolder, F.Cu at (238.7, -75.7)
- added R31: 1 kohm, Resistor_SMD:R_0603_1608Metric_Pad0.98x0.95mm_HandSolder, F.Cu at (238.7, -73.2)
- added R32: 1 kohm, Resistor_SMD:R_0603_1608Metric_Pad0.98x0.95mm_HandSolder, F.Cu at (238.7, -70.7)
- added R33: 1 kohm, Resistor_SMD:R_0603_1608Metric_Pad0.98x0.95mm_HandSolder, F.Cu at (230.0, -58.1)
- added R34: 1 kohm, Resistor_SMD:R_0603_1608Metric_Pad0.98x0.95mm_HandSolder, F.Cu at (230.0, -55.5)
- added R35: 1 kohm, Resistor_SMD:R_0603_1608Metric_Pad0.98x0.95mm_HandSolder, F.Cu at (230.0, -53.0)
- added R36: 1 kohm, Resistor_SMD:R_0603_1608Metric_Pad0.98x0.95mm_HandSolder, F.Cu at (230.0, -50.5)
- added R37: 1 kohm, Resistor_SMD:R_0603_1608Metric_Pad0.98x0.95mm_HandSolder, F.Cu at (230.0, -48.0)
- added R38: 1 kohm, Resistor_SMD:R_0603_1608Metric_Pad0.98x0.95mm_HandSolder, F.Cu at (230.0, -45.5)
- added R39: 1 kohm, Resistor_SMD:R_0603_1608Metric_Pad0.98x0.95mm_HandSolder, F.Cu at (230.0, -43.0)
- added R40: 1 kohm, Resistor_SMD:R_0603_1608Metric_Pad0.98x0.95mm_HandSolder, F.Cu at (234.3, -58.1)
- added R41: 1 kohm, Resistor_SMD:R_0603_1608Metric_Pad0.98x0.95mm_HandSolder, F.Cu at (234.3, -55.5)
- added R42: 1 kohm, Resistor_SMD:R_0603_1608Metric_Pad0.98x0.95mm_HandSolder, F.Cu at (234.3, -53.0)
- added R43: 1 kohm, Resistor_SMD:R_0603_1608Metric_Pad0.98x0.95mm_HandSolder, F.Cu at (234.3, -50.5)
- added R44: 1 kohm, Resistor_SMD:R_0603_1608Metric_Pad0.98x0.95mm_HandSolder, F.Cu at (234.3, -48.0)
- added R45: 1 kohm, Resistor_SMD:R_0603_1608Metric_Pad0.98x0.95mm_HandSolder, F.Cu at (234.3, -45.5)
- added R46: 1 kohm, Resistor_SMD:R_0603_1608Metric_Pad0.98x0.95mm_HandSolder, F.Cu at (234.3, -43.0)
- added R47: 1 kohm, Resistor_SMD:R_0603_1608Metric_Pad0.98x0.95mm_HandSolder, F.Cu at (238.7, -58.1)
- added R48: 1 kohm, Resistor_SMD:R_0603_1608Metric_Pad0.98x0.95mm_HandSolder, F.Cu at (238.7, -55.5)
- added R49: 1 kohm, Resistor_SMD:R_0603_1608Metric_Pad0.98x0.95mm_HandSolder, F.Cu at (238.7, -53.0)
- added R50: 1 kohm, Resistor_SMD:R_0603_1608Metric_Pad0.98x0.95mm_HandSolder, F.Cu at (238.7, -50.5)
- added R51: 5.1 kohm, Resistor_SMD:R_0612_1632Metric_Pad1.18x3.40mm_HandSolder, F.Cu at (245.0, -72.2)
- added R52: 5.1 kohm, Resistor_SMD:R_0612_1632Metric_Pad1.18x3.40mm_HandSolder, F.Cu at (245.0, -52.1)
- moved SW33 238.4 mm to (182.4, 127.8), turned to 48 degrees
- moved SW29 231.2 mm to (170.3, 149.7), turned to 76 degrees
- moved SW14 227.8 mm to (73.7, 77.6), turned to -20 degrees
- moved SW32 226.6 mm to (242.4, 75.7), turned to 20 degrees
- moved SW15 217.4 mm to (89.7, 89.5), turned to -20 degrees
- moved SW19 210.2 mm to (93.6, 113.7), turned to -20 degrees
- moved SW8 209.8 mm to (60.9, 57.9), turned to -20 degrees
- moved SW22 209.1 mm to (190.0, 98.1), turned to 20 degrees
- moved SW16 204.0 mm to (106.7, 97.9), turned to -20 degrees
- moved SW18 203.7 mm to (183.5, 80.1), turned to 20 degrees
- moved SW21 203.1 mm to (126.5, 149.7), turned to -76 degrees
- moved SW1 201.0 mm to (41.1, 44.2), turned to -15 degrees
- moved SW20 201.0 mm to (113.9, 127.8), turned to -48 degrees
- moved SW28 200.1 mm to (222.9, 77.3), turned to 20 degrees
- moved SW12 199.1 mm to (31.5, 80.9), turned to -15 degrees
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Connections:
- U4 pad 26: unconnected-(U4-PB13-Pad26) -> Net-(Q2-G)
- U8 pad 26: unconnected-(U8-PB13-Pad26) -> Net-(Q1-G)
