File: sichergo-left/sichergo-left.kicad_pcb (KiCad board)
At the start: 2 copper layers, 123.4 x 96.1 mm, 117 parts, among them J1 Conn_01x04_Pin, Q1 2N7002, SW1 SW_Push, SW10 SW_Push, SW11 SW_Push, SW12 SW_Push, SW13 SW_Push, SW14 SW_Push, SW15 SW_Push, SW16 SW_Push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

Commit message: Finish routing redesign
Routing:
- net GND: track 0.00 -> 23.2 mm, vias 0 -> 40
- net /KB_COL_4: track 132.3 -> 128.5 mm
- net /KB_COL_3: track 116.0 -> 112.7 mm
- net /KB_ROW_1: track 101.2 -> 99.4 mm
- net /KB_COL_2: track 122.3 -> 120.9 mm
- net +3V3: track 243.0 -> 241.8 mm
- net /KB_ROW_2: track 86.5 -> 85.3 mm
- net /KB_ROW_0: track 116.5 -> 115.4 mm
- net Net-(D36-A): track 13.7 -> 12.8 mm
- net /KB_COL_0: track 135.0 -> 134.1 mm
- net Net-(D29-A): track 13.8 -> 13.0 mm
- net Net-(Audio1-Pad3): track 19.4 -> 18.6 mm
- net Net-(U4-NRST): track 24.7 -> 24.0 mm
- net /MatrixL/LED_DRIVE: track 378.1 -> 377.5 mm
- net /VBUS: track 23.2 -> 23.8 mm
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