File: sichergo-left/MatrixL.kicad_sch (KiCad schematic)
At the start: 72 parts, among them SW1 SW_Push, SW10 SW_Push, SW11 SW_Push, SW12 SW_Push, SW13 SW_Push, SW14 SW_Push, SW15 SW_Push, SW16 SW_Push, SW19 SW_Push, SW20 SW_Push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

Commit message: Split design in two PCBs and remake layout
Parts:
- renumbered D69 to D10, D3 to D11, D8 to D12, D66 to D14, D65 to D15, D64 to D16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
